File: vfd.kicad_sch (KiCad schematic)
At the start: 45 parts, among them J1 I2C_IN, J2 I2C_OUT, Q1 BC857, Q2 BC847, Q3 BC857, Q4 BC847, U1 AP3012, U2 CH32V003F4U6, U3 AP3012, U4 74HCT541PW

Commit message: v0.2
Parts:
- removed R5: 1k, Resistor_SMD:R_0603_1608Metric, symbol Device:R_Small
- removed TP5, TP6, TP7, TP8, TP9: TestPoint, TestPoint:TestPoint_Pad_D1.5mm, symbol Connector:TestPoint
- added D3: LED, vfd:LED_0603_1608Metric, symbol vfd:LED
- added JP1: A0, vfd:SolderJumper-2_P1.3mm_Open_TrianglePad1.0x1.5mm, symbol vfd:Jumper_2_Open
- added JP2: A1, vfd:SolderJumper-2_P1.3mm_Open_TrianglePad1.0x1.5mm, symbol vfd:Jumper_2_Open
- added JP3: A2, vfd:SolderJumper-2_P1.3mm_Open_TrianglePad1.0x1.5mm, symbol vfd:Jumper_2_Open
- added JP4: A3, vfd:SolderJumper-2_P1.3mm_Open_TrianglePad1.0x1.5mm, symbol vfd:Jumper_2_Open
- added JP5: A4, vfd:SolderJumper-2_P1.3mm_Open_TrianglePad1.0x1.5mm, symbol vfd:Jumper_2_Open
- added N2: OSHW, Symbol:OSHW-Logo_5.7x6mm_SilkScreen, symbol vfd:Housing
- added R5: 270, vfd:R_0603_1608Metric, symbol vfd:R_Small
- C1, C2, C3, C4, C5, C6: footprint Capacitor_SMD:C_0603_1608Metric -> vfd:C_0603_1608Metric; symbol Device:C_Small -> vfd:C_Small
- D1, D2: footprint Diode_SMD:D_SOD-323 -> vfd:D_SOD-323; symbol Diode:1N5819WS -> vfd:1N5819WS
- J1, J2: footprint qwiic:1X04_1MM_RA_GND -> vfd:1X04_1MM_RA_GND; symbol qwiic:qwiic -> vfd:qwiic
- L1, L2: footprint power-circuit:Inductor_MSC20FC -> vfd:Inductor_MSC20FC; symbol Device:L_Small -> vfd:L_Small
- N1: value Housing -> Logo; footprint footprints:logo_nicolai -> vfd:logo_nicolai; symbol Mechanical:Housing -> vfd:Housing
- Q1, Q3: footprint Package_TO_SOT_SMD:SOT-23 -> vfd:SOT-23; symbol Transistor_BJT:BC857 -> vfd:BC857
- Q2, Q4: footprint Package_TO_SOT_SMD:SOT-23 -> vfd:SOT-23; symbol Transistor_BJT:BC847 -> vfd:BC847
- R1, R10, R11, R12, R13, R14, R2, R3, R4, R6, R7, R8, R9: footprint Resistor_SMD:R_0603_1608Metric -> vfd:R_0603_1608Metric; symbol Device:R_Small -> vfd:R_Small
- TP1, TP2, TP3, TP4: footprint TestPoint:TestPoint_Pad_D1.5mm -> vfd:TestPoint_Pad_D1.5mm; symbol Connector:TestPoint -> vfd:TestPoint
- U1, U3: footprint Package_TO_SOT_SMD:SOT-23-5 -> vfd:SOT-23-5; symbol Regulator_Switching:AP3012 -> vfd:AP3012
- U2: footprint Package_DFN_QFN:QFN-20-1EP_3x3mm_P0.4mm_EP1.65x1.65mm -> vfd:QFN-20-1EP_3x3mm_P0.4mm_EP1.65x1.65mm; symbol ch32v003:CH32V003F4U6 -> vfd:CH32V003F4U6
- U4: footprint Package_SO:TSSOP-20_4.4x6.5mm_P0.65mm -> vfd:TSSOP-20_4.4x6.5mm_P0.65mm; symbol 74xx:74HCT541 -> vfd:74HCT541
- U5: footprint hcs-12ss59t:HCS-12SS59T -> vfd:HCS-12SS59T; symbol hcs-12ss59t:HCS-12SS59T -> vfd:HCS-12SS59T
Connections:
- net +5V: now also Q1.2 (E), Q3.2 (E); no longer Q1.3 (C), Q3.3 (C)
- net CLK: now also U4.14 (Y4); no longer U4.15 (Y3)
- net CLK_A: now also U4.17 (Y1); no longer U4.18 (Y0)
- net CLK_A_LV: now also U4.3 (A1); no longer U4.2 (A0)
- net CLK_B: now also U4.18 (Y0); no longer U4.17 (Y1)
- net CLK_B_LV: now also U4.2 (A0); no longer U4.3 (A1)
- net CLK_LV: now also U4.6 (A4); no longer U4.5 (A3)
- net DIN: now also U4.13 (Y5); no longer U4.16 (Y2)
- net DIN_LV: now also U4.7 (A5); no longer U4.4 (A2)
- net F+: now also Q1.3 (C); no longer Q1.2 (E)
- net F-: now also Q3.3 (C); no longer Q3.2 (E)
- net GND: now also D3.1 (K), JP1.2 (B), JP2.2 (B), JP3.2 (B), JP4.2 (B), JP5.2 (B)
- net ~{CS_LV}: now also U4.5 (A3); no longer U4.7 (A5)
- net ~{CS}: now also U4.15 (Y3); no longer U4.13 (Y5)
- net ~{RST_LV}: now also U4.4 (A2); no longer U4.6 (A4)
- net ~{RST}: now also U4.16 (Y2); no longer U4.14 (Y4)
- net at U2.19 (PD5): now also JP2.1 (A)
- net at U2.17 (PD3): now also JP4.1 (A)
- net at U2.20 (PD6): now also JP1.1 (A)
- net at U2.18 (PD4): now also JP3.1 (A)
- net at U2.16 (PD2): now also JP5.1 (A)
- net ~{CPU_RST}: no longer names the net of U2.1 (PD7)
- net ~{CPU_RST}: now also R5.2
- new net: D3.2 (A), R5.1
Other:
- moved on the sheet: Q3

Commit message: Version 0.2 final
Parts:
- C1, C3, C4, C5: LCSC (none) -> C1592
- C2: LCSC (none) -> C282519
- C6: LCSC (none) -> C1683
- D1, D2: LCSC (none) -> C191023
- D3: LCSC (none) -> C264473
- J1, J2: Category Connectors -> (none); Field4 CONN-13694 -> (none); MPN SM04B-SRSS-TB -> (none); Manufacturer JST -> (none)
- JP1, JP2, JP3, JP4, JP5, N1, N2, TP1, TP2, TP3, TP4, U5: LCSC (none) -> -
- L1, L2: Part Ceaiya CRH201610S-100MT -> (none)
- Q1, Q3: LCSC C779725 -> C2139
- Q2, Q4: LCSC C779725 -> C475630
- R10, R12, R13, R9: LCSC (none) -> C21190
- R11, R8: LCSC (none) -> C25803
- R14: LCSC (none) -> C25981
- R3: LCSC (none) -> C25804
- R4: LCSC (none) -> C22984
- R5: LCSC (none) -> C22966
- R6: LCSC (none) -> C23186
- R7: LCSC (none) -> C23265
Changed lines of the file:
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@@
   (title_block
     (title "HCS-12SS59T VFD")
-    (date "2023-05-29")
-    (rev "0.1")
+    (date "2023-09-09")
+    (rev "0.2")
     (company "Nicolai Electronics")
   )
@@
       (effects (font (size 1.27 1.27)) hide)
     )
+    (property "LCSC" "C21190" (at 175.895 106.68 0)
+      (effects (font (size 1.27 1.27)) hide)
+    )
     (pin "1")
     (pin "2")
@@
       (effects (font (size 1.27 1.27)) hide)
     )
+    (property "LCSC" "C25981" (at 246.38 64.77 0)
+      (effects (font (size 1.27 1.27)) hide)
+    )
     (pin "1")
     (pin "2")
@@
       (effects (font (size 1.27 1.27)) hide)
     )
-    (property "Field4" "CONN-13694" (at 26.67 38.1 0)
-      (effects (font (size 1.524 1.524)) hide)
-    )
     (property "LCSC" "C160404" (at 29.21 49.53 0)
       (effects (font (size 1.27 1.27)) hide)
     )
-    (property "MPN" "SM04B-SRSS-TB" (at 29.21 49.53 0)
-      (effects (font (size 1.27 1.27)) hide)
-    )
-    (property "Manufacturer" "JST" (at 29.21 49.53 0)
-      (effects (font (size 1.27 1.27)) hide)
-    )
-    (property "Category" "Connectors" (at 29.21 49.53 0)
-      (effects (font (size 1.27 1.27)) hide)
-    )
     (pin "1")
     (pin "2")
@@
       (effects (font (size 1.27 1.27)) hide)
     )
+    (property "LCSC" "-" (at 104.14 21.59 0)
+      (effects (font (size 1.27 1.27)) hide)
+    )
     (pin "1")
     (pin "2")
@@
       (effects (font (size 1.27 1.27)) hide)
     )
+    (property "LCSC" "C1592" (at 109.855 106.68 0)
+      (effects (font (size 1.27 1.27)) hide)
+    )
     (pin "1")
     (pin "2")
@@
       (effects (font (size 1.27 1.27)) hide)
     )
-    (property "LCSC" "C779725" (at 207.645 91.44 0)
+    (property "LCSC" "C2139" (at 207.645 91.44 0)
       (effects (font (size 1.27 1.27)) hide)
     )
@@
       (effects (font (size 1.27 1.27)) hide)
     )
+    (property "LCSC" "C21190" (at 175.895 91.44 0)
+      (effects (font (size 1.27 1.27)) hide)
+    )
     (pin "1")
     (pin "2")
@@
       (effects (font (size 1.27 1.27)) hide)
     )
+    (property "LCSC" "C1683" (at 246.38 74.93 0)
+      (effects (font (size 1.27 1.27)) hide)
+    )
     (pin "1")
     (pin "2")
@@
       (effects (font (size 1.27 1.27)) hide)
     )
+    (property "LCSC" "C25803" (at 166.37 53.34 0)
+      (effects (font (size 1.27 1.27)) hide)
+    )
     (pin "1")
     (pin "2")
@@
       (effects (font (size 1.27 1.27)) hide)
     )
+    (property "LCSC" "C22966" (at 83.82 34.29 0)
+      (effects (font (size 1.27 1.27)) hide)
+    )
     (pin "1")
     (pin "2")
@@
       (effects (font (size 1.27 1.27)) hide)
     )
+    (property "LCSC" "C1592" (at 39.37 106.68 0)
+      (effects (font (size 1.27 1.27)) hide)
+    )
     (pin "1")
     (pin "2")
@@
       (effects (font (size 1.27 1.27)) hide)
     )
+    (property "LCSC" "-" (at 139.065 185.42 0)
+      (effects (font (size 1.27 1.27)) hide)
+    )
     (instances
       (project "vfd"
@@
       (effects (font (size 1.27 1.27)) hide)
     )
+    (property "LCSC" "C191023" (at 146.685 86.36 0)
+      (effects (font (size 1.27 1.27)) hide)
+    )
     (pin "1")
     (pin "2")
@@
       (effects (font (size 1.27 1.27)) hide)
     )
+    (property "LCSC" "-" (at 116.84 34.29 0)
+      (effects (font (size 1.27 1.27)) hide)
+    )
     (pin "1")
     (instances
@@
       (effects (font (size 1.27 1.27)) hide)
     )
+    (property "LCSC" "C23265" (at 146.685 100.33 0)
+      (effects (font (size 1.27 1.27)) hide)
+    )
     (pin "1")
     (pin "2")
@@
       (effects (font (size 1.27 1.27)) hide)
     )
+    (property "LCSC" "C21190" (at 215.265 106.68 0)
+      (effects (font (size 1.27 1.27)) hide)
+    )
     (pin "1")
     (pin "2")
@@
       (effects (font (size 1.27 1.27)) hide)
     )
+    (property "LCSC" "-" (at 156.845 184.785 0)
+      (effects (font (size 1.27 1.27)) hide)
+    )
     (instances
       (project "vfd"
@@
       (effects (font (size 1.27 1.27)) hide)
     )
+    (property "LCSC" "C25803" (at 176.53 53.34 0)
+      (effects (font (size 1.27 1.27)) hide)
+    )
     (pin "1")
     (pin "2")
@@
       (effects (font (size 1.27 1.27)) hide)
     )
+    (property "LCSC" "C23186" (at 141.605 106.68 0)
+      (effects (font (size 1.27 1.27)) hide)
+    )
     (pin "1")
     (pin "2")
@@
       (effects (font (size 1.27 1.27)) hide)
     )
+    (property "LCSC" "C25804" (at 71.12 106.68 0)
+      (effects (font (size 1.27 1.27)) hide)
+    )
     (pin "1")
     (pin "2")
@@
       (effects (font (size 1.27 1.27)) hide)
     )
+    (property "LCSC" "-" (at 106.68 21.59 0)
+      (effects (font (size 1.27 1.27)) hide)
+    )
     (pin "1")
     (pin "2")
@@
       (effects (font (size 1.27 1.27)) hide)
     )
+    (property "LCSC" "-" (at 101.6 21.59 0)
+      (effects (font (size 1.27 1.27)) hide)
+    )
     (pin "1")
     (pin "2")
@@
       (effects (font (size 1.27 1.27)) hide)
     )
+    (property "LCSC" "C191023" (at 76.2 86.36 0)
+      (effects (font (size 1.27 1.27)) hide)
+    )
     (pin "1")
     (pin "2")
@@
       (effects (font (size 1.27 1.27)) hide)
     )
-    (property "LCSC" "C779725" (at 207.645 106.68 0)
+    (property "LCSC" "C475630" (at 207.645 106.68 0)
       (effects (font (size 1.27 1.27)) hide)
     )
@@
       (effects (font (size 1.27 1.27)) hide)
     )
+    (property "LCSC" "-" (at 269.24 53.34 0)
+      (effects (font (size 1.27 1.27)) hide)
+    )
     (pin "1")
     (pin "10")
@@
       (effects (font (size 1.27 1.27)) hide)
     )
+    (property "LCSC" "C1592" (at 153.035 106.68 0)
+      (effects (font (size 1.27 1.27)) hide)
+    )
     (pin "1")
     (pin "2")
@@
       (effects (font (size 1.27 1.27)) hide)
     )
+    (property "LCSC" "-" (at 114.3 36.83 0)
+      (effects (font (size 1.27 1.27)) hide)
+    )
     (pin "1")
     (instances
@@
       (effects (font (size 1.27 1.27)) hide)
     )
-    (property "Field4" "CONN-13694" (at 52.07 38.1 0)
-      (effects (font (size 1.524 1.524)) hide)
-    )
     (property "LCSC" "C160404" (at 49.53 49.53 0)
       (effects (font (size 1.27 1.27)) hide)
     )
-    (property "MPN" "SM04B-SRSS-TB" (at 49.53 49.53 0)
-      (effects (font (size 1.27 1.27)) hide)
-    )
-    (property "Manufacturer" "JST" (at 49.53 49.53 0)
-      (effects (font (size 1.27 1.27)) hide)
-    )
-    (property "Category" "Connectors" (at 49.53 49.53 0)
-      (effects (font (size 1.27 1.27)) hide)
-    )
     (pin "1")
     (pin "2")
@@
       (effects (font (size 1.27 1.27)) hide)
     )
-    (property "LCSC" "C779725" (at 183.515 91.44 0)
+    (property "LCSC" "C2139" (at 183.515 91.44 0)
       (effects (font (size 1.27 1.27)) hide)
     )
@@
       (effects (font (size 1.27 1.27)) hide)
     )
-    (property "Part" "Ceaiya CRH201610S-100MT" (at 58.42 86.36 90)
-      (effects (font (size 1.27 1.27)) hide)
-    )
     (property "LCSC" "C520204" (at 58.42 86.36 90)
       (effects (font (size 1.27 1.27)) hide)
@@
       (effects (font (size 1.27 1.27)) hide)
     )
+    (property "LCSC" "-" (at 99.06 21.59 0)
+      (effects (font (size 1.27 1.27)) hide)
+    )
     (pin "1")
     (pin "2")
@@
       (effects (font (size 1.27 1.27)) hide)
     )
-    (property "Part" "Ceaiya CRH201610S-100MT" (at 128.905 86.36 90)
-      (effects (font (size 1.27 1.27)) hide)
-    )
     (property "LCSC" "C520204" (at 128.905 86.36 90)
       (effects (font (size 1.27 1.27)) hide)
@@
       (effects (font (size 1.27 1.27)) hide)
     )
+    (property "LCSC" "C1592" (at 82.55 106.68 0)
+      (effects (font (size 1.27 1.27)) hide)
+    )
     (pin "1")
     (pin "2")
@@
       (effects (font (size 1.27 1.27)) hide)
     )
-    (property "LCSC" "C779725" (at 183.515 106.68 0)
+    (property "LCSC" "C475630" (at 183.515 106.68 0)
       (effects (font (size 1.27 1.27)) hide)
     )
@@
       (effects (font (size 1.27 1.27)) hide)
     )
+    (property "LCSC" "-" (at 138.43 35.56 0)
+      (effects (font (size 1.27 1.27)) hide)
+    )
     (pin "1")
     (instances
@@
       (effects (font (size 1.27 1.27)) hide)
     )
+    (property "LCSC" "-" (at 135.89 35.56 0)
+      (effects (font (size 1.27 1.27)) hide)
+    )
     (pin "1")
     (instances
@@
       (effects (font (size 1.27 1.27)) hide)
     )
+    (property "LCSC" "C22984" (at 76.2 100.33 0)
+      (effects (font (size 1.27 1.27)) hide)
+    )
     (pin "1")
     (pin "2")
@@
       (effects (font (size 1.27 1.27)) hide)
     )
+    (property "LCSC" "C21190" (at 215.265 91.44 0)
+      (effects (font (size 1.27 1.27)) hide)
+    )
     (pin "1")
     (pin "2")
@@
       (effects (font (size 1.27 1.27)) hide)
     )
+    (property "LCSC" "C264473" (at 77.47 34.29 0)
+      (effects (font (size 1.27 1.27)) hide)
+    )
     (pin "1")
     (pin "2")
@@
       (effects (font (size 1.27 1.27)) hide)
     )
+    (property "LCSC" "-" (at 96.52 21.59 0)
+      (effects (font (size 1.27 1.27)) hide)
+    )
     (pin "1")
     (pin "2")
@@
       (effects (font (size 1.27 1.27)) hide)
     )
+    (property "LCSC" "C282519" (at 73.66 57.15 0)
+      (effects (font (size 1.27 1.27)) hide)
+    )

Commit message: Make inductor pads bigger, make vfd pads and holes larger
Parts:
- L1, L2: footprint vfd:Inductor_MSC20FC -> vfd:Inductor_201610

Commit message: Revision 1.0 final
Parts:
- added J3: I2C_HDR, Connector_PinHeader_2.54mm:PinHeader_1x04_P2.54mm_Vertical, symbol Connector_Generic:Conn_01x04
- added N3: Logo, vfd:logo_nicolai, symbol vfd:Housing
- TP1: value TestPoint -> SWIO
- TP2: value TestPoint -> EXT
- TP3: value TestPoint -> GND
- TP4: value TestPoint -> 3.3v
Connections:
- net +3.3V: now also J3.3 (Pin_3)
- net GND: now also J3.4 (Pin_4)
- net SCL: now also J3.1 (Pin_1)
- net SDA: now also J3.2 (Pin_2)
Other:
- moved on the sheet: C4, C5, D2, L2, Q1, Q2, Q3, Q4, R10, R12, R13, R6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
